File: EGACard.kicad_sch (KiCad schematic)
At the start: 48 parts, among them U14 S04, U16 LS27, U17 LS32, U18 74LS74, U26 LS04, U27 LS11, U30 LS32, U47 LS04, U5 LS10, U6 LS00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

Commit message: U5, U6 -> S, not LS logic
Parts:
- U5: value LS10 -> S10
- U6: value LS00 -> S00
Changed lines of the file:
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@@
       (effects (font (size 1.27 1.27)))
     )
-    (property "Value" "LS00" (at 35.56 120.65 0)
+    (property "Value" "S00" (at 35.56 120.65 0)
       (effects (font (size 1.27 1.27)))
     )
@@
       (effects (font (size 1.27 1.27)))
     )
-    (property "Value" "LS10" (at 24.13 120.65 0)
+    (property "Value" "S10" (at 24.13 120.65 0)
       (effects (font (size 1.27 1.27)))
     )
