File: Sheet3.kicad_sch (KiCad schematic)
At the start: 10 parts, among them U17 LS32, U19 LS374, U20 LS174, U22 LS374, U26 LS04, U32 CRT CNTL, U42 LS374, U5 LS10, U52 LS374, U6 LS00

Commit message: U5, U6 -> S, not LS logic
Parts:
- U5: value LS10 -> S10
- U6: value LS00 -> S00
Changed lines of the file:
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@@
       (effects (font (size 1.27 1.27)))
     )
-    (property "Value" "LS00" (at 124.46 31.75 0)
+    (property "Value" "S00" (at 124.46 31.75 0)
       (effects (font (size 1.27 1.27)))
     )
@@
       (effects (font (size 1.27 1.27)))
     )
-    (property "Value" "LS10" (at 124.46 15.24 0)
+    (property "Value" "S10" (at 124.46 15.24 0)
       (effects (font (size 1.27 1.27)))
     )
@@
       (effects (font (size 1.27 1.27)))
     )
-    (property "Value" "LS10" (at 165.1 54.61 0)
+    (property "Value" "S10" (at 165.1 54.61 0)
       (effects (font (size 1.27 1.27)))
     )
@@
       (effects (font (size 1.27 1.27)))
     )
-    (property "Value" "LS00" (at 138.43 46.99 0)
-      (effects (font (size 1.27 1.27)))
-    )
+    (property "Value" "S00" (at 138.43 46.99 0)
+      (effects (font (size 1.27 1.27)))
+    )
