File: Sheet5.kicad_sch (KiCad schematic)
At the start: 8 parts, among them U18 74LS74, U26 LS04, U27 LS11, U42 LS374, U5 LS10, U6 LS00

Commit message: U5, U6 -> S, not LS logic
Parts:
- U5: value LS10 -> S10
- U6: value LS00 -> S00
Changed lines of the file:
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@@
       (effects (font (size 1.27 1.27)))
     )
-    (property "Value" "LS00" (at 163.83 146.05 0)
+    (property "Value" "S00" (at 163.83 146.05 0)
       (effects (font (size 1.27 1.27)))
     )
@@
       (effects (font (size 1.27 1.27)))
     )
-    (property "Value" "LS10" (at 215.8917 76.2 0)
+    (property "Value" "S10" (at 215.8917 76.2 0)
       (effects (font (size 1.27 1.27)))
     )
@@
       (effects (font (size 1.27 1.27)))
     )
-    (property "Value" "LS00" (at 163.83 157.48 0)
+    (property "Value" "S00" (at 163.83 157.48 0)
       (effects (font (size 1.27 1.27)))
     )
